Commit message: update edu_450 other files

File: src/edu_450/urdf/edu_450.urdf (robot description, URDF)
Before this commit: robot edu_450, 5 links, 4 joints
Links:
- link drone_link: mass 0.94206 -> 1.1106
Joints:
- joint rotor1_joint: origin xyz=0.15689 -0.15689 0.080664 rpy=0 0 0 -> xyz=0.15631 -0.15652 0.060014 rpy=0 0 0
- joint rotor2_joint: origin xyz=-0.15689 0.15689 0.080664 rpy=0 0 0 -> xyz=-0.15748 0.15727 0.060014 rpy=0 0 0
- joint rotor3_joint: axis -0.061628 -0.061628 0.99619 -> -0.0616284167162217 -0.0616284167162192 0.996194698091745; origin xyz=0.15689 0.15689 0.080664 rpy=0 0 0 -> xyz=0.15630948387772 0.157266901286137 0.0600141878263292 rpy=0 0 0
- joint rotor4_joint: origin xyz=-0.15689 -0.15689 0.080664 rpy=0 0 0 -> xyz=-0.15748 -0.15652 0.060014 rpy=0 0 0
